File: HW/transceiver/mcu.sch (KiCad schematic (older format))
At the start: 23 parts, among them K8 SAM_JTAG, X1 FA-238V-12MHZ

Commit message: PCB of transceiver designed.
Parts:
- C14, C15, C16, C17, C18, C19, C20, C21, C22, C23, C24: footprint ~ -> Capacitors_SMD:C_0603; symbol C -> C-RESCUE-modballoon
- DD4: footprint (none) -> Housings_QFP:LQFP-64_10x10mm_Pitch0.5mm
- K8: footprint ~ -> Pin_Headers:Pin_Header_Straight_2x10
- L6, L7: footprint ~ -> Capacitors_SMD:C_0805
- R10, R4, R5, R6, R7, R8, R9: footprint ~ -> Resistors_SMD:R_0603; symbol R -> R-RESCUE-modballoon
- X1: footprint (none) -> Balloln_pretty:crystal_FA238-TSX3225; symbol FA-238V-12MHZ -> FA-238V-12MHz
Other:
- moved on the sheet: C14, C15, C16, C17, C18, C19, C20, C21, C22, C23, C24, DD4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
