File: HW/transceiver/Modem.sch (KiCad schematic (older format))
At the start: 86 parts, among them X2 7Q-26.000MBN-T

Commit message: PCB of transceiver designed.
Parts:
- C25, C26, C27, C28, C29, C30, C31, C33, C35, C37, C38, C40, C41, C42, C43, C44, C45, C46, C47, C48, C49, C50, C51, C52, C53, C54, C55, C56, C57, C58, C59, C60, C61, C62, C63, C64, C65, C66, C67, C68, C69, C70, C71, C72, C73, C74, C75: footprint ~ -> Capacitors_SMD:C_0603; symbol C -> C-RESCUE-modballoon
- C32, C34, C36, C39: value 100n -> M1; footprint ~ -> Capacitors_SMD:C_0603; symbol C -> C-RESCUE-modballoon
- DD10: footprint ~ -> TO_SOT_Packages_SMD:SOT89-3_Housing
- DD5: footprint (none) -> Balloln_pretty:QFN-20-1EP_4x4mm_Pitch0.5mm; symbol SI4463 -> si4463
- DD6: footprint ~ -> Balloln_pretty:UQFN-16-1EP_3x3mm_Pitch0.5mm
- DD7: footprint ~ -> TO_SOT_Packages_SMD:SC-70-5
- DD8: footprint ~ -> Balloln_pretty:SAW
- DD9: footprint ~ -> TO_SOT_Packages_SMD:SOT-23-6
- L10, L11, L12, L13, L14, L15, L16, L17, L24, L27, L8, L9: footprint ~ -> Capacitors_SMD:C_0805
- L18, L19, L20, L21, L22, L23, L25, L26, L29, L31, L33: footprint 0603 -> Capacitors_SMD:C_0603
- L28, L30, L32: footprint 0306 -> Capacitors_SMD:C_0603
- R11, R12: footprint ~ -> Resistors_SMD:R_0603; symbol R -> R-RESCUE-modballoon
- X2: footprint (none) -> Balloln_pretty:crystal_FA238-TSX3225
