File: HW/transceiver/modballoon.kicad_pcb (KiCad board)
At the start: 4 copper layers, 101.1 x 50.3 mm, 153 parts, among them K1 CONN_6, K2 CONN_10, K3 CONN_6, K4 CONN_6, K5 SMA, K6 SMA, K7 HE10-20, K8 SAM_JTAG, M1 CONN_01X01, M2 CONN_01X01, M3 CONN_01X01, M4 CONN_01X01, M5 CONN_01X01, M6 CONN_01X01, M7 CONN_01X01, M8 CONN_01X01, X1 FA-238V-12MHZ, X2 7Q-26.000MBN-T

Commit message: PCB generate production data
Other:
- rule pad_to_mask_clearance: 0 -> 0.2
Changed lines of the file:
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@@
     (pad_size 1.5 1.5)
     (pad_drill 0.6)
-    (pad_to_mask_clearance 0)
+    (pad_to_mask_clearance 0.2)
+    (solder_mask_min_width 0.2)
     (aux_axis_origin 0 0)
     (visible_elements 7FFFFFFF)
     (pcbplotparams
-      (layerselection 0x00030_80000001)
+      (layerselection 0x010f0_80000007)
       (usegerberextensions false)
       (excludeedgelayer true)
@@
       (outputformat 1)
       (mirror false)
-      (drillshape 1)
+      (drillshape 0)
       (scaleselection 1)
-      (outputdirectory ""))
+      (outputdirectory CAM_PROFI/))
   )
   (net 0 "")
